Commit message: slam toolbox ok

File: diff_drive_robot/urdf/robot_core.xacro (robot description, xacro)
@@ -2,4 +2,10 @@
 <robot xmlns:xacro="http://www.ros.org/wiki/xacro" >
   <xacro:include filename="inertial_macros.xacro" />
+  <link name="base_footprint"/>
+  <joint name="base_link_joint" type="fixed">
+    <parent link="base_footprint"/>
+    <child link="base_link"/>
+    <origin xyz="0 0 0"/>
+  </joint>
   <!-- Base link -->
   <link name="base_link"/>
