Commit message: Add navigation and SLAM configuration files for Jetson Rover
- Created nav2_params_base.yaml with parameters for AMCL, costmaps, planners, and behavior servers.
- Added spatio_temporal_voxel_layer.yaml and voxel_layer.yaml for costmap layers.
- Implemented rtabmap_navigation.launch.py and rtabmap_navigation.launch.copy for RTAB-Map integration.
- Updated rtabmap.launch.py and rtabmap_slam.launch.py for improved SLAM functionality.
- Introduced yaml_join.py script to merge YAML configuration files for dynamic layer integration.
- Enhanced launch files to support namespace and simulation configurations.

File: diff_drive_robot/urdf/dabai_dcw.urdf.xacro (robot description, xacro)
@@ -45,5 +45,5 @@
     visualize:=true
     enable_collision:=false">
-    <link name="${prefix}camera_link">
+    <link name="${prefix}depth_cam_link">
       <visual>
         <origin xyz="0 0 0" rpy="0 0 0"/>
@@ -72,5 +72,5 @@
     <joint name="${prefix}${camera_name}_joint" type="fixed">
       <parent link="${prefix}base_link"/>
-      <child link="${prefix}camera_link" />
+      <child link="${prefix}depth_cam_link" />
       <origin xyz="${xyz_offset}" rpy="${rpy_offset}"/>
     </joint>

File: diff_drive_robot/urdf/robot.urdf.xacro (robot description, xacro)
@@ -21,5 +21,5 @@
     <!-- <xacro:include filename="ros_control.xacro" /> -->
     <xacro:include filename="lidar.xacro" />
-    <xacro:include filename="$(find diff_drive_robot)/urdf/imu.xacro"/>
+    <xacro:include filename="$(find diff_drive_robot)/urdf/imu_1500.xacro"/>
     <xacro:include filename="$(find diff_drive_robot)/urdf/dabai_dcw.urdf.xacro"/>
     <xacro:imu_sensor
