Commit message: motion and imu change over;wait test

File: diff_drive_robot/urdf/1.urdf (robot description, URDF)
Before this commit: robot diff_drive_robot, 7 links, 6 joints
Links:
- added link imu_link, mass 0.031; visual box size=0.03899 0.03785 0.01338
- link front_castor_wheel: geometry collision sphere radius=0.055; visual sphere radius=0.055
- link rear_castor_wheel: geometry collision sphere radius=0.055; visual sphere radius=0.055
Joints:
- added joint imu_joint: type fixed, parent chassis, child imu_link, origin xyz=0 0 0.006 rpy=0 0 0
- joint chassis_joint: origin xyz=0 0 0.34199999999999997 -> xyz=0 0 0.346
- joint front_castor_wheel_joint: origin xyz=0.299 0 0.051 -> xyz=0.295 0 0.055
- joint laser_joint: origin xyz=0.1 0 0.291 rpy=0 0 0 -> xyz=0.28 0 0.353 rpy=0 0 0
- joint rear_castor_wheel_joint: origin xyz=-0.299 0 0.051 -> xyz=-0.295 0 0.055

File: diff_drive_robot/urdf/lidar.xacro (robot description, xacro)
@@ -6,5 +6,5 @@
      <parent link="chassis"/>
      <child link="laser_frame"/>
-     <origin xyz="0.1 0 ${chassis_link_h/2+laser_width/2}" rpy="0 0 0"/>
+     <origin xyz="0.28 0 0.353" rpy="0 0 0"/>
    </joint>
    <link name="laser_frame">

File: diff_drive_robot/urdf/robot.urdf.xacro (robot description, xacro)
@@ -7,15 +7,26 @@
     <xacro:if value="${machine == 'JetRover_Mecanum'}">
     </xacro:if> -->
+    <xacro:arg name="prefix" default=""/>
+    <xacro:arg name="use_gazebo" default="false"/>
     <xacro:property name="chassis_link_l"        value="0.7"/>
     <xacro:property name="chassis_link_w"        value="0.52"/>
     <xacro:property name="chassis_link_h"        value="0.582"/>
     <xacro:property name="wheel_base"        value="0.593"/>
-    <xacro:property name="chassis_high"        value="0.051"/>
+    <xacro:property name="chassis_high"        value="0.055"/>
     <xacro:property name="wheel_diameter"        value="0.2"/>
     <xacro:property name="wheel_width"        value="0.04"/>
-    <xacro:property name="wheel_interval"        value="0.04"/>
+    <xacro:property name="wheel_interval"        value="0.047"/>
     <xacro:include filename="robot_core.xacro" />
     <!-- <xacro:include filename="gazebo_control.xacro" /> -->
-    <xacro:include filename="ros_control.xacro" />
+    <!-- <xacro:include filename="ros_control.xacro" /> -->
     <xacro:include filename="lidar.xacro" />
+    <xacro:include filename="$(find diff_drive_robot)/urdf/imu.xacro"/>
+    <xacro:imu_sensor
+      prefix="$(arg prefix)"
+      parent="chassis"
+      frame_id="imu"
+      xyz_offset="0 0 0.006"
+      rpy_offset="0 0 0"
+      update_rate="15.0"
+      topic_name="imu/data"/>
 </robot>

Commit message: Update URDF and configuration for camera integration; adjust lidar joint parameters and enhance navigation costmap settings

File: diff_drive_robot/urdf/1.urdf (robot description, URDF)
Before this commit: robot diff_drive_robot, 8 links, 7 joints
Links:
- added link base_footprint
- added link camera_depth_optical_frame, mass 0.072; visual box size=0.02 0.08 0.02
Joints:
- added joint base_link_joint: type fixed, parent base_footprint, child base_link, origin xyz=0 0 0
- added joint cam_1_joint: type fixed, parent chassis, child camera_depth_optical_frame, origin xyz=0.105 0 0.05 rpy=0 -0.50 0
- joint imu_joint: origin xyz=0 0 0.006 rpy=0 0 0 -> xyz=0.34 0 -0.15599999999999997 rpy=0 0 0

File: diff_drive_robot/urdf/lidar.xacro (robot description, xacro)
@@ -4,7 +4,7 @@
     <xacro:property name="laser_width"        value="0.04"/>
    <joint name="laser_joint" type="fixed">
-     <parent link="chassis"/>
+     <parent link="base_link"/>
      <child link="laser_frame"/>
-     <origin xyz="0.28 0 0.353" rpy="0 0 0"/>
+     <origin xyz="0.28 0 0.41" rpy="0 0 0"/>
    </joint>
    <link name="laser_frame">

File: diff_drive_robot/urdf/robot.urdf.xacro (robot description, xacro)
@@ -22,4 +22,5 @@
     <xacro:include filename="lidar.xacro" />
     <xacro:include filename="$(find diff_drive_robot)/urdf/imu.xacro"/>
+    <xacro:include filename="$(find diff_drive_robot)/urdf/dabai_dcw.urdf.xacro"/>
     <xacro:imu_sensor
       prefix="$(arg prefix)"
@@ -30,3 +31,8 @@
       update_rate="15.0"
       topic_name="imu/data"/>
+    <xacro:dabai_dcw
+      prefix="$(arg prefix)"
+      camera_name="dabai_dcw"
+      xyz_offset="0.28 0 0.51"
+      rpy_offset="0 0 0"/>
 </robot>

Commit message: add fire distance

File: diff_drive_robot/urdf/1.urdf (robot description, URDF)
Before this commit: robot diff_drive_robot, 10 links, 9 joints
Links:
- removed link camera_depth_optical_frame
- added link camera_link, mass 0.072; visual box size=0.02 0.08 0.02
- added link left_hk_camera_optical_frame, mass 0.072; visual box size=0.05 0.08 0.05
- added link right_hk_camera_optical_frame, mass 0.072; visual box size=0.05 0.08 0.05
Joints:
- removed joint cam_1_joint
- added joint astra_pro_plus_joint: type fixed, parent base_link, child camera_link, origin xyz=0.24 -0.02 0.51 rpy=0 0 0
- added joint left_hk_camera_joint: type fixed, parent base_link, child left_hk_camera_optical_frame, origin xyz=0.27 0.165 0.423 rpy=0 0 0
- added joint right_hk_camera_joint: type fixed, parent base_link, child right_hk_camera_optical_frame, origin xyz=0.27 -0.132 0.423 rpy=0 0 0
- joint imu_joint: origin xyz=0.34 0 -0.15599999999999997 rpy=0 0 0 -> xyz=0.16 -0.1 -0.291 rpy=0 0 0
- joint laser_joint: origin xyz=0.28 0 0.353 rpy=0 0 0 -> xyz=0.28 0 0.41 rpy=0 0 0; parent chassis -> base_link

File: diff_drive_robot/urdf/hk_ir_camera.urdf.xacro (robot description, xacro)
@@ -4,5 +4,5 @@
   <xacro:macro name="hk_ir_camera" params="
     prefix:=''
-    camera_name:='hk_ir_camera'
+    camera_name:='hk_camera'
     parent:='base_link'
     xyz_offset:='0.30 0.25 0.22'
@@ -45,5 +45,5 @@
     visualize:=true
     enable_collision:=false">
-    <link name="${prefix}hk_ir_camera_link">
+    <link name="${prefix}${camera_name}_optical_frame">
       <visual>
         <origin xyz="0 0 0" rpy="0 0 0"/>
@@ -71,6 +71,6 @@
     </link>
     <joint name="${prefix}${camera_name}_joint" type="fixed">
-      <parent link="${prefix}base_link"/>
-      <child link="${prefix}hk_ir_camera_link" />
+      <parent link="base_link"/>
+      <child link="${prefix}${camera_name}_optical_frame" />
       <origin xyz="${xyz_offset}" rpy="${rpy_offset}"/>
     </joint>

File: diff_drive_robot/urdf/lidar.xacro (robot description, xacro)
@@ -6,5 +6,5 @@
      <parent link="base_link"/>
      <child link="laser_frame"/>
-     <origin xyz="0.28 0 0.41" rpy="0 0 0"/>
+     <origin xyz="0.28 0 0.315" rpy="0 0 0"/>
    </joint>
    <link name="laser_frame">

File: diff_drive_robot/urdf/robot.urdf.xacro (robot description, xacro)
@@ -38,4 +38,26 @@
       rpy_offset="0 0 0"/> -->
       <xacro:astra_pro_plus/>
-      <xacro:hk_ir_camera/>
+      <xacro:hk_ir_camera
+        prefix="left_"
+        xyz_offset="0.27 0.164 0.423"
+      />
+      <xacro:hk_ir_camera
+        prefix="right_"
+        xyz_offset="0.27 -0.13 0.423"
+      />
+    <joint name="stereo_ir_camera_joint" type="fixed">
+      <parent link="base_link"/>  <!-- 或者其他合适的父link -->
+      <child link="stereo_ir_camera"/> <!-- 虚拟的 -->
+      <origin xyz="0.27 0.017 0.423" rpy="0 0 0"/>  <!-- 根据实际安装位置调整 -->
+    </joint>
+    <link name="stereo_ir_camera">
+      <visual>
+        <geometry>
+          <box size="0 0 0"/>  <!-- 双相机支架的大致尺寸 -->
+        </geometry>
+        <material name="black">
+          <color rgba="0.2 0.2 0.2 1"/>
+        </material>
+      </visual>
+    </link>
 </robot>
