Commit message: cartographer slam and nav ok

File: diff_drive_robot/urdf/imu_1500.xacro (robot description, xacro)
@@ -4,5 +4,5 @@
     <xacro:macro name="imu_sensor" params="
         prefix:=''
-        parent:='chassis'
+        parent:='base_link'
         frame_id:='imu'
         xyz_offset:='0.34 0 0'
@@ -51,5 +51,5 @@
             <parent link="${prefix}${parent}"/>
             <child link="${prefix}${frame_id}_link" />
-            <origin xyz="0.16 -0.1 ${-chassis_link_h/2}" rpy="${rpy_offset}"/>
+            <origin xyz="0.16 -0.1 0.055" rpy="${rpy_offset}"/>
         </joint>
         <gazebo reference="${prefix}${frame_id}_link">

File: diff_drive_robot/urdf/robot.urdf.xacro (robot description, xacro)
@@ -26,7 +26,7 @@
     <xacro:imu_sensor
       prefix="$(arg prefix)"
-      parent="chassis"
+      parent="base_link"
       frame_id="imu"
-      xyz_offset="0 0 0.006"
+      xyz_offset="0.16 -0.1 0.055"
       rpy_offset="0 0 0"
       update_rate="15.0"
